File: board/cape.brd (EAGLE design)
At the start: 100 x 80 mm, 17 parts

Commit message: Finished schematic and routing.
Parts:
- removed C2: 100uF 35V, rcl:E5-10,5
- removed C3: 0.1uF, rcl:C0603
- removed C4: 0.47uF, rcl:C0603
- removed D1: 1N5400, diode:DO201-15
- removed U$4: LM2585, Twitterbot:TO263
- added 5VREG: LM2576-5.0WT, national-semiconductor:TO263-5
- added BATT_S, VCC_S: ADM1191, custom:MSOP-10
- added C6: 1000uF, rcl:175TMP-0808
- added C7: 100uF, rcl:153CLV-0605
- added D2: 40V 3A Schottky, diode:DO-214AC
- added IC1: CAT24C256WI, microchip:SO-08
- added L1: 100uH, Twitterbot:INDUCTOR
- added R5: 0.02, resistor:R0603
- added R6: 10k, rcl:R0603
- added S1: SWS002, smd-special:SMS-002
- added WP: PTR1TP10R, testpad:TP10R
- C1: value 680uF 16V (1189-1150-ND) -> 0.1uF; device rcl:E5-10,5 -> rcl:C0603
- F1: device fuse:LITTLEFUSE -> Twitterbot:2920
- R4: value 2k -> 0.02; device rcl:R0603 -> resistor:R0603
- moved U$2 144.9 mm to (44.5, 66.0), turned to 270 degrees
- moved R3 136.4 mm to (41.3, 44.5), turned to 180 degrees
- moved F1 130.5 mm to (12.1, 80.6), flipped to the bottom
- moved DISP 129.0 mm to (45.7, 55.9), turned to 180 degrees
- moved U$3 124.1 mm to (45.7, 44.5)
- moved R2 121.2 mm to (38.7, 67.3), turned to 180 degrees
- moved TTL 119.8 mm to (45.7, 34.3), turned to 270 degrees
- moved R1 117.1 mm to (38.7, 64.8), turned to 180 degrees
- moved R4 103.7 mm to (13.4, 73.4)
- moved PWR 91.0 mm to (45.1, 76.2), turned to 90 degrees
- moved C1 89.6 mm to (38.7, 40.3), turned to 180 degrees
- moved U$1 68.6 mm to (0.00, 0.00)
Connections:
- net N$6 renamed SW
- removed net N$10: R4.1, U$4.1
- removed net N$4: R2.2, U$1.46
- removed net N$5: R1.2, U$1.45
- removed net N$7: C1.+, D1.C
- new net GRN_LED: R2.2, U$1.45
- new net I2C1_SCL: BATT_S.6, U$1.63, VCC_S.6
- new net I2C1_SDA: BATT_S.7, U$1.64, VCC_S.7
- new net I2C2_SCL: IC1.6, U$1.65
- new net I2C2_SDA: IC1.5, U$1.66
- new net N$11: IC1.1, S1.1
- new net N$12: IC1.2, S1.2
- new net N$13: 5VREG.4, C6.+, L1.2, R5.1, VCC_S.1, VCC_S.8
- new net N$17: IC1.7, R6.1, WP.TP
- new net N$8: 5VREG.2, D2.C, L1.1
- new net RED_LED: R1.2, U$1.46
- net 12V_FUSE: now also 5VREG.1, BATT_S.2, C7.+, R4.2; no longer C2.+, C3.1, F1.2, U$4.5
- net GND: now also 5VREG.3, 5VREG.5, BATT_S.4, BATT_S.8, BATT_S.9, C1.2, C6.-, C7.-, D2.A, IC1.4, VCC_S.4, VCC_S.9; no longer C2.-, C3.2, C4.2, U$4.3, U$4.TAB
- net N$9: now also BATT_S.1, F1.2, R4.1; no longer C4.1, R4.2
- net VCC: now also C1.1, IC1.3, IC1.8, R6.2, S1.3, S1.4
- net VDD_5V: now also R5.2, VCC_S.2
Routing:
- net VCC: track 0.00 -> 94.0 mm, vias 0 -> 1
- net I2C1_SCL: track 0.00 -> 79.4 mm, vias 0 -> 2
- net I2C1_SDA: track 0.00 -> 77.6 mm, vias 0 -> 2
- net VDD_5V: track 0.00 -> 54.9 mm
- net SW: track 0.00 -> 50.1 mm, vias 0 -> 1
- net N$13: track 0.00 -> 47.1 mm
- net RED_LED: track 0.00 -> 40.2 mm, vias 0 -> 1
- net GRN_LED: track 0.00 -> 36.6 mm, vias 0 -> 1
- net 12VDC: track 0.00 -> 31.6 mm
- net I2C2_SCL: track 0.00 -> 17.0 mm
- net I2C2_SDA: track 0.00 -> 15.6 mm
- net MOSI: track 0.00 -> 13.4 mm
- net N$9: track 0.00 -> 12.6 mm, vias 0 -> 1
- net 12V_FUSE: track 0.00 -> 12.4 mm
- net N$8: track 0.00 -> 11.1 mm
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- added copper zone on layer 1, net GND
- added copper zone on layer 16, net GND
Other:
- board size 100 x 80 mm -> 54.6 x 71.8 mm
- board text added: "0 0 0x54 0 1 0x55 1 0 0x56 1 1 0x57"
- board text added: "0x60"
- board text added: "0x78"
- board text added: "7-30VDC <=3A"
- board text added: "A0"
- board text added: "A1"
- board text added: "A1 A0 ADDR"
- board text added: "CS"
- board text added: "GND"
- board text added: "GRN"
- board text added: "MOSI"
- board text added: "NC"
- board text added: "NO"
- board text added: "RED"
- board text added: "RXI"
- board text added: "SCLK"
- board text added: "TXO"
- board text added: "VCC"
