File: board/cape.brd (EAGLE design)
At the start: 54.6 x 71.8 mm, 24 parts, among them IC1 CAT24C256WI

Commit message: Added project information and logos to board.
Parts:
- added U$4: (no value), ohw-logo:OSHW_FILLX350_NOTEXT
Other:
- board text added: "http://i3detroit.com/wi/index.php?title=I3TwitterBot Andrew G. Meyer (agmlego)"
- board text added: "i3Twitterbot"
