File: board/cape.sch (EAGLE design)
At the start: 17 parts

Commit message: Finished schematic and routing.
Parts:
- removed C2: 100uF 35V, rcl:CPOL-USE5-10.5
- removed C3: 0.1uF, rcl:C-USC0603
- removed C4: 0.47uF, rcl:C-USC0603
- removed D1: 1N5400, diode:1N5400
- removed U$4: LM2585, Twitterbot:LM2585
- added 5VREG: LM2576-5.0WT, national-semiconductor:LM2596S
- added BATT_S, VCC_S: ADM1191, custom:ADM1191
- added C6: 1000uF, rcl:CPOL-US175TMP-0808
- added C7: 100uF, rcl:CPOL-US153CLV-0605
- added D2: 40V 3A Schottky, diode:DIODE-DO-214AC
- added IC1: CAT24C256WI, microchip:24AA01SN
- added L1: 100uH, Twitterbot:INDUCTOR
- added R5: 0.02, resistor:R-US_R0603
- added R6: 10k, rcl:R-US_R0603
- added S1: SWS002, smd-special:SWS002
- added WP: PTR1TP10R, testpad:PTR1TP10R
- C1: value 680uF 16V (1189-1150-ND) -> 0.1uF; device rcl:CPOL-USE5-10.5 -> rcl:C-USC0603
- F1: device fuse:FUSELITTLEFUSE -> Twitterbot:FUSE2920; DIGIKEY (none) -> F2875CT-ND
- R4: value 2k -> 0.02; device rcl:R-US_R0603 -> resistor:R-US_R0603; DIGIKEY (none) -> WSLL-.02CT-ND
Connections:
- net N$6 renamed SW
- removed net N$10: R4.1, U$4.COMP
- removed net N$4: R2.2, U$1.GPIO2_7
- removed net N$5: R1.2, U$1.GPIO2_6
- removed net N$7: C1.+, D1.C
- new net GRN_LED: R2.2, U$1.GPIO2_6
- new net I2C1_SCL: BATT_S.SCL, U$1.I2C1_SCL, VCC_S.SCL
- new net I2C1_SDA: BATT_S.SDA, U$1.I2C1_SDA, VCC_S.SDA
- new net I2C2_SCL: IC1.SCL, U$1.I2C2_SCL
- new net I2C2_SDA: IC1.SDA, U$1.I2C2_SDA
- new net N$11: IC1.A0, S1.1
- new net N$12: IC1.A1, S1.2
- new net N$13: 5VREG.FB, C6.+, L1.2, R5.1, VCC_S.A0, VCC_S.VCC
- new net N$17: IC1.WP, R6.1, WP.TP
- new net N$8: 5VREG.OUT, D2.C, L1.1
- new net RED_LED: R1.2, U$1.GPIO2_7
- new net VDD_5V: R5.2, U$1.VDD_5V@1, U$1.VDD_5V@2, VCC_S.SENSE
- net 12V_FUSE: now also 5VREG.VIN, BATT_S.SENSE, C7.+, R4.2; no longer C2.+, C3.1, F1.2, U$4.VIN
- net GND: now also 5VREG.!ON!/OFF, 5VREG.GND, BATT_S.A0, BATT_S.A1, BATT_S.GND, C1.2, C6.-, C7.-, D2.A, IC1.GND, VCC_S.A1, VCC_S.GND; no longer C2.-, C3.2, C4.2, U$4.GND
- net N$9: now also BATT_S.VCC, F1.2, R4.1; no longer C4.1, R4.2
- net VCC: now also C1.1, IC1.A2, IC1.VCC, R6.2, S1.3, S1.4
Other:
- note added: "0x60"
- note added: "0x78"
- moved on the sheet: PWR, R4

Commit message: Altered board to as-built greenwiring, fixing confusion on SPI1_D0/SPI1_D1 and moving the switch from a necessary boot-configuration pin to a free one.
Connections:
- removed net MOSI: DISP.MOSI, U$1.SPI1_DO
- new net N$4: DISP.MOSI, U$1.SPI1_DI
- net SW: now also U$1.GPIO0_7; no longer U$1.GPIO2_9
Changed lines of the file:
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@@
 <setting verticaltext="up"/>
 </settings>
-<grid distance="0.1" unitdist="inch" unit="inch" style="lines" multiple="1" display="no" altdistance="0.01" altunitdist="inch" altunit="inch"/>
+<grid distance="0.05" unitdist="inch" unit="inch" style="lines" multiple="1" display="no" altdistance="0.01" altunitdist="inch" altunit="inch"/>
 <layers>
 <layer number="1" name="Top" color="4" fill="1" visible="no" active="no"/>
@@
 </segment>
 </net>
-<net name="MOSI" class="0">
-<segment>
-<pinref part="DISP" gate="G$1" pin="MOSI"/>
-<pinref part="U$1" gate="G$1" pin="SPI1_DO"/>
-<wire x1="-119.38" y1="27.94" x2="-101.6" y2="27.94" width="0.1524" layer="91"/>
-</segment>
-</net>
 <net name="SCLK" class="0">
 <segment>
@@
 <segment>
 <pinref part="R3" gate="G$1" pin="2"/>
-<wire x1="-3.81" y1="85.09" x2="-21.59" y2="85.09" width="0.1524" layer="91"/>
-<wire x1="-21.59" y1="85.09" x2="-21.59" y2="76.2" width="0.1524" layer="91"/>
-<pinref part="U$1" gate="G$1" pin="GPIO2_9"/>
-<wire x1="-21.59" y1="76.2" x2="-45.72" y2="76.2" width="0.1524" layer="91"/>
+<wire x1="-3.81" y1="85.09" x2="-33.02" y2="85.09" width="0.1524" layer="91"/>
+<wire x1="-33.02" y1="85.09" x2="-33.02" y2="12.7" width="0.1524" layer="91"/>
+<pinref part="U$1" gate="G$1" pin="GPIO0_7"/>
+<wire x1="-33.02" y1="12.7" x2="-45.72" y2="12.7" width="0.1524" layer="91"/>
 </segment>
 </net>
@@
 </segment>
 </net>
+<net name="N$4" class="0">
+<segment>
+<pinref part="DISP" gate="G$1" pin="MOSI"/>
+<wire x1="-119.38" y1="27.94" x2="-106.68" y2="27.94" width="0.1524" layer="91"/>
+<wire x1="-106.68" y1="27.94" x2="-106.68" y2="29.21" width="0.1524" layer="91"/>
+<pinref part="U$1" gate="G$1" pin="SPI1_DI"/>
+<wire x1="-106.68" y1="29.21" x2="-45.72" y2="29.21" width="0.1524" layer="91"/>
+<wire x1="-45.72" y1="29.21" x2="-45.72" y2="27.94" width="0.1524" layer="91"/>
+</segment>
+</net>
